File: BrainDamage.kicad_pcb (KiCad board)
At the start: 2 copper layers, 90 x 90 mm, 25 parts, among them CON1 AVR-ISP-10, IC1 ATMEGA328P-A, P1 CONN_01X03, P10 CONN_01X03, P11 CONN_01X03, P12 CONN_01X03, P13 CONN_01X03, P14 CONN_01X03, P15 CONN_01X03, P16 CONN_01X03, P17 CONN_01X03, P2 CONN_01X03, P3 CONN_01X03, P4 CONN_01X03, P5 CONN_01X03, P6 CONN_01X03, P7 CONN_01X03, P8 CONN_01X08, P9 CONN_01X03, SW1 SW_PUSH, U1 PCA9685-TSSOP

Commit message: Add files via upload
Parts:
- added J1: TEST_2P, Connectors:GS2, F.Cu at (196.0, 52.0)
- added J2: TEST_2P, Connectors:GS2, F.Cu at (198.0, 52.0)
- added J3: TEST_2P, Connectors:GS2, F.Cu at (200.0, 52.0)
- added J4: TEST_2P, Connectors:GS2, F.Cu at (202.0, 52.0)
- added J5: TEST_2P, Connectors:GS2, F.Cu at (204.0, 52.0)
- added J6: TEST_2P, Connectors:GS2, F.Cu at (186.9, 65.5)
- added J7: FTDI, Pin_Headers:Pin_Header_Angled_1x05_Pitch2.54mm, F.Cu at (191.6, 71.0)
- added J8: Bluetooth, Pin_Headers:Pin_Header_Straight_1x04_Pitch2.54mm, B.Cu at (163.0, 63.9)
- added R3: 10K, Resistors_SMD:R_0805_HandSoldering, F.Cu at (203.3, 70.2)
- added R4: 10K, Resistors_SMD:R_0805_HandSoldering, F.Cu at (192.0, 66.8)
- added R5: 10K, Resistors_SMD:R_0805_HandSoldering, F.Cu at (187.7, 68.0)
- added R6: 20K, Resistors_SMD:R_0805_HandSoldering, F.Cu at (158.5, 63.0)
- added R7: 20K, Resistors_SMD:R_0805_HandSoldering, F.Cu at (171.0, 76.5)
- added R8: 10K, Resistors_SMD:R_0805_HandSoldering, F.Cu at (158.5, 65.0)
- added R9: 10K, Resistors_SMD:R_0805_HandSoldering, F.Cu at (166.5, 78.0)
- added REF**: Test_Point_Pad_1.0x1.0mm, Connectors_TestPoints:Test_Point_Pad_1.0x1.0mm, F.Cu at (200.5, 86.5)
- added REF**: Test_Point_THTPad_4.0x4.0mm_Drill2.0mm, Connectors_TestPoints:Test_Point_THTPad_4.0x4.0mm_Drill2.0mm, F.Cu at (219.0, 25.0)
- added REF**: Test_Point_Pad_1.0x1.0mm, Connectors_TestPoints:Test_Point_Pad_1.0x1.0mm, F.Cu at (199.5, 85.0)
- added REF**: Test_Point_Pad_1.0x1.0mm, Connectors_TestPoints:Test_Point_Pad_1.0x1.0mm, F.Cu at (198.5, 86.5)
- added REF**: Test_Point_Pad_1.0x1.0mm, Connectors_TestPoints:Test_Point_Pad_1.0x1.0mm, F.Cu at (197.5, 85.0)
- added REF**: Test_Point_Pad_1.0x1.0mm, Connectors_TestPoints:Test_Point_Pad_1.0x1.0mm, F.Cu at (201.5, 85.0)
- added REF**: Test_Point_Pad_1.0x1.0mm, Connectors_TestPoints:Test_Point_Pad_1.0x1.0mm, F.Cu at (196.5, 86.5)
- added REF**: Test_Point_THTPad_4.0x4.0mm_Drill2.0mm, Connectors_TestPoints:Test_Point_THTPad_4.0x4.0mm_Drill2.0mm, F.Cu at (181.0, 25.0)
- added REF**: Test_Point_THTPad_4.0x4.0mm_Drill2.0mm, Connectors_TestPoints:Test_Point_THTPad_4.0x4.0mm_Drill2.0mm, F.Cu at (181.0, 41.0)
- added REF**: Test_Point_THTPad_4.0x4.0mm_Drill2.0mm, Connectors_TestPoints:Test_Point_THTPad_4.0x4.0mm_Drill2.0mm, F.Cu at (219.0, 41.0)
- added X1: CRYSTAL_SMD, Crystals:Resonator_SMD_muRata_SFSKA-3pin_7.9x3.8mm_HandSoldering, F.Cu at (172.0, 84.5)
- CON1: footprint Pin_Headers:Pin_Header_Straight_2x05_Pitch2.54mm_SMD -> Pin_Headers:Pin_Header_Straight_2x05_Pitch2.54mm; moved to B.Cu
- P1, P10, P11, P12, P13, P14, P15, P16, P17, P2, P3, P4, P5, P6, P7, P9: footprint Pin_Headers:Pin_Header_Straight_1x03_Pitch1.27mm -> Pin_Headers:Pin_Header_Straight_1x03_Pitch2.54mm; moved to B.Cu
- P8: footprint Pin_Headers:Pin_Header_Angled_1x08_Pitch1.27mm -> Pin_Headers:Pin_Header_Angled_1x08_Pitch2.54mm; moved to B.Cu
- moved D1 49.6 mm to (227.5, 85.0), turned to 90 degrees
- moved R1 46.1 mm to (230.0, 85.0), turned to 270 degrees
- moved P17 26.6 mm to (172.5, 47.0), turned to 90 degrees
- moved P1 26.6 mm to (227.5, 47.0), turned to 270 degrees
- moved P16 21.9 mm to (227.5, 71.5), turned to 270 degrees
- moved P7 21.3 mm to (172.5, 71.5), turned to 90 degrees
- moved P2 20.5 mm to (227.5, 50.5), turned to 270 degrees
- moved P15 20.4 mm to (172.5, 50.5), turned to 90 degrees
- moved P8 19.2 mm to (222.7, 94.2)
- moved P14 16.0 mm to (227.5, 68.0), turned to 270 degrees
- moved P9 15.4 mm to (172.5, 68.0), turned to 90 degrees
- moved P3 14.7 mm to (227.5, 54.0), turned to 270 degrees
- moved P13 14.6 mm to (172.5, 54.0), turned to 90 degrees
- moved CON1 14.2 mm to (197.9, 98.5)
- moved P6 11.0 mm to (227.5, 64.5), turned to 270 degrees
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Connections:
- net Net-(IC1-Pad32) renamed /PD2
- CON1 pad 2: +3V3 -> +5V
- IC1 pad 1: /PIN6 -> /TXB
- IC1 pad 10: /PIN4 -> /PD6
- IC1 pad 11: Net-(IC1-Pad11) -> /PD7
- IC1 pad 12: /B1 -> /PB0
- IC1 pad 13: /PIN1 -> /PB1
- IC1 pad 14: /PIN2 -> /PB2
- IC1 pad 2: Net-(IC1-Pad2) -> /RXB
- IC1 pad 23: /A0 -> /PC0
- IC1 pad 24: /A1 -> /PC1
- IC1 pad 25: /A2 -> /PC2
- IC1 pad 26: /A3 -> /PC3
- IC1 pad 9: /PIN5 -> /PD5
- P1 pad 1: /LED0 -> /LED7
- P1 pad 2: +3V3 -> +5V
- P10 pad 1: /LED10 -> /LED13
- P10 pad 2: +3V3 -> +5V
- P11 pad 1: /LED11 -> /LED12
- P11 pad 2: +3V3 -> +5V
- P12 pad 1: /LED12 -> /LED11
- P12 pad 2: +3V3 -> +5V
- P13 pad 1: /LED13 -> /LED10
- P13 pad 2: Net-(P13-Pad2) -> +5V
- P14 pad 1: /LED6 -> /LED1
- P14 pad 2: +3V3 -> +5V
- P15 pad 1: /LED14 -> /LED9
- P15 pad 2: +3V3 -> +5V
- P16 pad 1: /LED7 -> /LED0
- P16 pad 2: +3V3 -> +5V
- P17 pad 1: /LED15 -> /LED8
- P17 pad 2: +3V3 -> +5V
- P2 pad 1: /LED1 -> /LED6
- P2 pad 2: +3V3 -> +5V
- P3 pad 1: /LED2 -> /LED5
- P3 pad 2: +3V3 -> +5V
- P4 pad 1: /LED3 -> /LED4
- P4 pad 2: +3V3 -> +5V
- P5 pad 1: /LED4 -> /LED3
- P5 pad 2: +3V3 -> +5V
- P6 pad 1: /LED5 -> /LED2
- P6 pad 2: Net-(P6-Pad2) -> +5V
- P7 pad 1: /LED8 -> /LED15
- P7 pad 2: +3V3 -> +5V
- P8 pad 1: /SCL -> /ADC6
- P8 pad 2: /SDA -> /ADC7
- P8 pad 3: /A3 -> /PC0
- P8 pad 4: /A2 -> /PC1
- P8 pad 5: /A1 -> /PC2
- P8 pad 6: /A0 -> /PC3
- P8 pad 7: /ADC7 -> GND
- P8 pad 8: /ADC6 -> +5V
- P9 pad 1: /LED9 -> /LED14
- P9 pad 2: +3V3 -> +5V
- U1 pad 1: Net-(U1-Pad1) -> /A0
- U1 pad 2: Net-(U1-Pad2) -> /A1
- U1 pad 23: Net-(U1-Pad23) -> /OE
- U1 pad 24: Net-(U1-Pad24) -> /A5
- U1 pad 25: Net-(U1-Pad25) -> GND
- U1 pad 3: Net-(U1-Pad3) -> /A2
- U1 pad 4: Net-(U1-Pad4) -> /A3
- U1 pad 5: Net-(U1-Pad5) -> /A4
Routing:
- net +5V: track 0.00 -> 394.2 mm
- net GND: track 2.99 -> 89.5 mm
- net (no net): track 0.00 -> 39.3 mm
- net /TXB: track 0.00 -> 36.8 mm
- net /ADC7: track 0.00 -> 26.3 mm
- net /PC3: track 0.00 -> 25.6 mm
- net /XTAL2: track 0.00 -> 24.9 mm
- net /ADC6: track 0.00 -> 24.7 mm
- net /PC2: track 0.00 -> 24.2 mm
- net /PC0: track 0.00 -> 23.9 mm
- net /RXB: track 0.00 -> 23.6 mm
- net /PC1: track 0.00 -> 23.2 mm
- net /XTAL1: track 0.00 -> 22.4 mm
- net /TX: track 0.00 -> 21.4 mm
- net /RX: track 0.00 -> 19.1 mm
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Other:
- board size 90 x 90 mm -> 100 x 100 mm
- net class Default: clearance 0.2 -> 0.25
- rule trace_clearance: 0.2 -> 0.25
- board text added: "!floating ground!"
- board text added: "@ecco1996 2018"
- board text added: "FTDI"
- board text added: "IRIS Robotics MV27T v0.1"

Commit message: Add files via upload
Parts:
- moved J1 22.4 mm to (210.0, 69.5), turned to 180 degrees
- moved J2 22.4 mm to (212.0, 69.5), turned to 180 degrees
- moved J3 22.4 mm to (214.0, 69.5), turned to 180 degrees
- moved J4 22.4 mm to (216.0, 69.5), turned to 180 degrees
- moved J5 22.4 mm to (218.0, 69.5), turned to 180 degrees
Routing:
- net GND: track 89.5 -> 56.0 mm
- net +5V: track 394.2 -> 372.8 mm
- net /A0: track 18.7 -> 7.62 mm
- net /A1: track 17.2 -> 10.3 mm
- net /A2: track 15.6 -> 12.6 mm
- net /A4: track 14.4 -> 17.1 mm
Other:
- board text added: "Address"

Commit message: Add files via upload
Parts:
- removed J7: FTDI, Pin_Headers:Pin_Header_Angled_1x05_Pitch2.54mm
- removed R6: 20K, Resistors_SMD:R_0805_HandSoldering
- removed R8: 10K, Resistors_SMD:R_0805_HandSoldering
- removed the REF** at (219.0, 25.0)
- removed the REF** at (181.0, 25.0)
- removed the REF** at (181.0, 41.0)
- removed the REF** at (219.0, 41.0)
- added BATT+: Measurement_Point_Square-SMD-Pad_Big, Measurement_Points:Measurement_Point_Square-SMD-Pad_Big, F.Cu at (218.0, 26.0)
- added C1: C, Capacitors_SMD:C_Trimmer_Murata_TZB4-A, F.Cu at (165.5, 46.5)
- added C2: C, Capacitors_SMD:C_Trimmer_Murata_TZB4-A, F.Cu at (235.4, 81.4)
- added C3: C, Capacitors_SMD:C_0805_HandSoldering, F.Cu at (188.5, 81.5)
- added C4: 1n, Capacitors_SMD:C_0805_HandSoldering, F.Cu at (172.5, 82.5)
- added C5: 1n, Capacitors_SMD:C_0805_HandSoldering, F.Cu at (213.0, 87.0)
- added C6: C, Capacitors_SMD:C_0805_HandSoldering, F.Cu at (212.8, 93.6)
- added GND: Measurement_Point_Square-SMD-Pad_Big, Measurement_Points:Measurement_Point_Square-SMD-Pad_Big, F.Cu at (210.0, 26.0)
- added J10: Conn_01x02, RC-Battery-Connectors:XT-60_male, B.Cu at (230.4, 40.4)
- added J9: USB_OTG, Connectors:USB_Mini-B, F.Cu at (187.3, 100.5)
- added REF**: Pin_Header_Straight_1x01_Pitch1.00mm, Pin_Headers:Pin_Header_Straight_1x01_Pitch1.00mm, F.Cu at (175.0, 31.0)
- added REF**: Pin_Header_Straight_1x01_Pitch1.00mm, Pin_Headers:Pin_Header_Straight_1x01_Pitch1.00mm, F.Cu at (225.0, 31.0)
- added REF**: Pin_Header_Straight_1x01_Pitch1.00mm, Pin_Headers:Pin_Header_Straight_1x01_Pitch1.00mm, F.Cu at (225.0, 51.0)
- added REF**: Pin_Header_Straight_1x01_Pitch1.00mm, Pin_Headers:Pin_Header_Straight_1x01_Pitch1.00mm, F.Cu at (175.0, 51.0)
- added U2: CH340G, Housings_SSOP:SOP-16_4.4x10.4mm_Pitch1.27mm, F.Cu at (180.5, 88.0)
- added U3: AP1117-50, TO_SOT_Packages_SMD:SOT-223-3Lead_TabPin2, F.Cu at (215.0, 100.2)
- added X2: CRYSTAL_SMD, Crystals:Resonator_SMD_muRata_SFSKA-3pin_7.9x3.8mm_HandSoldering, F.Cu at (172.0, 89.0)
- moved J8 23.5 mm to (181.4, 78.5), turned to 270 degrees
- moved R5 21.2 mm to (208.8, 70.5)
- moved R7 19.2 mm to (190.2, 75.5)
- moved X1 17.5 mm to (189.0, 88.8)
- moved R9 17.0 mm to (183.2, 81.5), turned to 0 degrees
- moved S0 5.70 mm to (231.0, 76.0)
- moved S1 5.70 mm to (231.0, 72.5)
- moved S2 5.70 mm to (231.0, 69.0)
- moved S3 5.70 mm to (231.0, 65.5)
- moved S4 5.70 mm to (231.0, 62.0)
- moved S5 5.70 mm to (231.0, 58.5)
- moved S6 5.70 mm to (231.0, 55.0)
- moved S7 5.70 mm to (231.0, 51.5)
- moved P8 5.37 mm to (222.7, 99.6)
- moved S10 5.00 mm to (169.5, 58.0)
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- renumbered P16 to S0, P14 to S1, P13 to S10, P12 to S11, P11 to S12, P10 to S13, P9 to S14, P7 to S15, P6 to S2, P5 to S3, P4 to S4, P3 to S5, P2 to S6, P1 to S7, P17 to S8, P15 to S9
Connections:
- J8 pad 1: Net-(J8-Pad1) -> +5V
Routing:
- net /BATT+: track 0.00 -> 85.2 mm, vias 0 -> 1
- net /TXB: track 36.8 -> 13.3 mm
- net /RXB: track 23.6 -> 4.46 mm
- net +5V: track 372.8 -> 354.1 mm
- net /RX: track 19.1 -> 35.4 mm
- net Net-(J9-Pad3): track 0.00 -> 16.0 mm
- net Net-(J9-Pad2): track 0.00 -> 14.5 mm
- net GND: track 56.0 -> 69.2 mm, vias 0 -> 15
- net /TX: track 21.4 -> 33.9 mm
- net /XTAL1: track 22.4 -> 10.5 mm
- net Net-(U2-Pad7): track 0.00 -> 9.06 mm
- net /XTAL2: track 24.9 -> 16.4 mm
- net Net-(C4-Pad1): track 0.00 -> 7.61 mm
- net /LED15: track 27.8 -> 35.1 mm
- net Net-(J8-Pad4): track 10.3 -> 3.08 mm
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- added copper zone on B.Cu, net GND
Other:
- board size 100 x 100 mm -> 100 x 85 mm
- board text added: "IRIS Robotics MV27T v1"
- board text removed: "!floating ground!"
- board text removed: "@ecco1996 2018"
- board text removed: "FTDI"
- board text removed: "IRIS Robotics MV27T v0.1"

Commit message: Add files via upload
Parts:
- added J11: Conn_01x04, Pin_Headers:Pin_Header_Straight_1x04_Pitch2.54mm, F.Cu at (183.3, 48.1)
- added J12: Conn_01x04, Pin_Headers:Pin_Header_Straight_1x04_Pitch2.54mm, F.Cu at (206.2, 48.1)
- added J7: 15A, Pin_Headers:Pin_Header_Angled_1x05_Pitch2.54mm, F.Cu at (193.5, 50.7)
- added REF**: Pin_Header_Straight_2x04_Pitch2.54mm, Pin_Headers:Pin_Header_Straight_2x04_Pitch2.54mm, F.Cu at (226.0, 87.0)
- P8: footprint Pin_Headers:Pin_Header_Angled_1x08_Pitch2.54mm -> Pin_Headers:Pin_Header_Straight_1x08_Pitch2.54mm; moved to F.Cu
- moved J10 3.45 mm to (227.0, 41.0)
- moved D1 2.69 mm to (226.5, 82.5)
- moved R1 2.69 mm to (229.0, 82.5)
- turned P8 to 180 degrees
Connections:
- IC1 pad 11: /PD7 -> /PG
Routing:
- net +5V: track 354.1 -> 401.7 mm
- net /PG: track 0.00 -> 36.9 mm, vias 0 -> 1
- net GND: track 69.2 -> 79.3 mm, vias 15 -> 17
- net /BATT+: track 85.2 -> 94.5 mm
- net /PD7: track 4.37 -> 2.92 mm
Other:
- board text added: "@ecco1996 2018"

Commit message: Add files via upload
Parts:
- J7: footprint Pin_Headers:Pin_Header_Angled_1x05_Pitch2.54mm -> Pin_Headers:Pin_Header_Straight_1x05_Pitch2.54mm
- moved C3 5.27 mm to (183.2, 81.0), turned to 180 degrees
- moved R9 5.20 mm to (188.3, 81.5), turned to 180 degrees
- moved REF** 0.60 mm to (225.4, 87.0)
Connections:
- REF** pad 1: /PD7 -> /PG
Routing:
- net /RESET: track 30.2 -> 39.6 mm, vias 0 -> 2
- net Net-(J8-Pad4): track 3.08 -> 7.62 mm
- net GND: track 79.3 -> 83.6 mm, vias 17 -> 19
- net /PG: track 36.9 -> 39.9 mm
- net /PD7: track 2.92 -> 0.00 mm
- net (no net): track 39.8 -> 39.3 mm, vias 1 -> 0

Commit message: Add files via upload
Routing:
- net /RESET: track 39.6 -> 72.9 mm
- net GND: track 83.6 -> 85.4 mm, vias 19 -> 15
Other:
- net class Default: via_dia 0.8 -> 1; via_drill 0.4 -> 0.6

Commit message: Add files via upload
Parts:
- added C7: 1n, Capacitors_SMD:C_0805_HandSoldering, F.Cu at (194.4, 91.6)
- moved BATT+ 2.00 mm to (218.0, 24.0)
- moved GND 2.00 mm to (210.0, 24.0)
Routing:
- net /RESET: track 72.9 -> 42.0 mm
- net Net-(C7-Pad1): track 0.00 -> 21.4 mm
- net GND: track 85.4 -> 87.5 mm, vias 15 -> 16
- net /BATT+: track 94.5 -> 96.5 mm

Commit message: Add files via upload
Parts:
- added R6: 10K, Resistors_SMD:R_0805_HandSoldering, F.Cu at (197.9, 96.0)
Routing:
- net +5V: track 401.7 -> 407.0 mm
- net /RESET: track 42.0 -> 42.8 mm
Changed lines of the file:
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@@
     (thickness 1.6)
     (drawings 32)
-    (tracks 536)
+    (tracks 540)
     (zones 0)
-    (modules 66)
+    (modules 67)
     (nets 72)
   )
@@
     )
   )
+  (module Resistors_SMD:R_0805_HandSoldering (layer F.Cu)
+    (at 197.9 96)
+    (descr "Resistor SMD 0805, hand soldering")
+    (tags "resistor 0805")
+    (attr smd)
+    (fp_text reference R6 (at 0 -1.7) (layer F.SilkS)
+      (effects (font (size 1 1) (thickness 0.15)))
+    )
+    (fp_text value 10K (at 0 1.75) (layer F.Fab)
+      (effects (font (size 1 1) (thickness 0.15)))
+    )
+    (fp_line (start 2.35 0.9) (end -2.35 0.9) (layer F.CrtYd) (width 0.05))
+    (fp_line (start 2.35 0.9) (end 2.35 -0.9) (layer F.CrtYd) (width 0.05))
+    (fp_line (start -2.35 -0.9) (end -2.35 0.9) (layer F.CrtYd) (width 0.05))
+    (fp_line (start -2.35 -0.9) (end 2.35 -0.9) (layer F.CrtYd) (width 0.05))
+    (fp_line (start -0.6 -0.88) (end 0.6 -0.88) (layer F.SilkS) (width 0.12))
+    (fp_line (start 0.6 0.88) (end -0.6 0.88) (layer F.SilkS) (width 0.12))
+    (fp_line (start -1 -0.62) (end 1 -0.62) (layer F.Fab) (width 0.1))
+    (fp_line (start 1 -0.62) (end 1 0.62) (layer F.Fab) (width 0.1))
+    (fp_line (start 1 0.62) (end -1 0.62) (layer F.Fab) (width 0.1))
+    (fp_line (start -1 0.62) (end -1 -0.62) (layer F.Fab) (width 0.1))
+    (fp_text user %R (at 0 0) (layer F.Fab)
+      (effects (font (size 0.5 0.5) (thickness 0.075)))
+    )
+    (pad 2 smd rect (at 1.35 0) (size 1.5 1.3) (layers F.Cu F.Paste F.Mask)
+      (net 2 /RESET))
+    (pad 1 smd rect (at -1.35 0) (size 1.5 1.3) (layers F.Cu F.Paste F.Mask)
+      (net 18 +5V))
+    (model ${KISYS3DMOD}/Resistors_SMD.3dshapes/R_0805.wrl
+      (at (xyz 0 0 0))
+      (scale (xyz 1 1 1))
+      (rotate (xyz 0 0 0))
+    )
+  )
   (gr_line (start 221.5 29) (end 178.5 29) (layer F.SilkS) (width 0.2))
   (gr_line (start 174 106) (end 150 64) (layer Margin) (width 0.1))
@@
   (segment (start 196.35 65.775) (end 197.15 65.775) (width 0.25) (layer F.Cu) (net 1))
   (segment (start 197.15 65.775) (end 197.15 65.799999) (width 0.25) (layer F.Cu) (net 1))
+  (segment (start 199.25 96) (end 200.25 96) (width 0.25) (layer F.Cu) (net 2))
+  (segment (start 200.25 96) (end 200.75 95.5) (width 0.25) (layer F.Cu) (net 2))
+  (segment (start 200.75 95.5) (end 201.396781 95.5) (width 0.25) (layer F.Cu) (net 2))
+  (segment (start 201.4 93.7) (end 200.500008 93.7) (width 0.25) (layer B.Cu) (net 2))
+  (segment (start 200.500008 93.7) (end 200.5 93.700008) (width 0.25) (layer B.Cu) (net 2))
   (segment (start 195.3 88.3) (end 194.4 89.2) (width 0.25) (layer F.Cu) (net 2))
   (segment (start 194.4 89.2) (end 194.4 90.35) (width 0.25) (layer F.Cu) (net 2))
-  (via (at 200.5 95.100022) (size 1) (drill 0.6) (layers F.Cu B.Cu) (net 2))
+  (via (at 201.4 93.7) (size 1) (drill 0.6) (layers F.Cu B.Cu) (net 2))
   (segment (start 196.9 90.100008) (end 200.5 93.700008) (width 0.25) (layer B.Cu) (net 2))
-  (segment (start 200.5 94.534337) (end 200.5 95.100022) (width 0.25) (layer B.Cu) (net 2))
   (segment (start 196.9 88.3) (end 196.9 90.100008) (width 0.25) (layer F.Cu) (net 2))
   (segment (start 201.396781 95.5) (end 201.39676 95.500021) (width 0.25) (layer F.Cu) (net 2))
-  (segment (start 200.899999 95.500021) (end 200.5 95.100022) (width 0.25) (layer F.Cu) (net 2))
-  (segment (start 200.5 93.700008) (end 200.5 94.534337) (width 0.25) (layer B.Cu) (net 2))
-  (segment (start 201.39676 95.500021) (end 200.899999 95.500021) (width 0.25) (layer F.Cu) (net 2))
   (via (at 196.9 90.100008) (size 1) (drill 0.6) (layers F.Cu B.Cu) (net 2))
   (segment (start 203 98.5) (end 203 97.1) (width 0.25) (layer F.Cu) (net 2))
@@
   (segment (start 194.346008 87.346008) (end 195.3 88.3) (width 0.25) (layer F.Cu) (net 2))
   (segment (start 195.3 88.3) (end 196.9 88.3) (width 0.25) (layer F.Cu) (net 2))
-  (segment (start 202 83.5) (end 202.5 84) (width 0.25) (layer F.Cu) (net 3))
   (segment (start 202.5 86.683805) (end 199.98575 89.198055) (width 0.25) (layer F.Cu) (net 3))
+  (segment (start 197.92 97.4) (end 197.92 98.5) (width 0.25) (layer F.Cu) (net 3))
   (segment (start 202.5 84) (end 202.5 86.683805) (width 0.25) (layer F.Cu) (net 3))
+  (segment (start 202 83.5) (end 202.5 84) (width 0.25) (layer F.Cu) (net 3))
   (segment (start 202 82.25) (end 202 83.5) (width 0.25) (layer F.Cu) (net 3))
-  (segment (start 199.98575 89.198055) (end 199.98575 93.31425) (width 0.25) (layer F.Cu) (net 3))
-  (segment (start 199.98575 93.31425) (end 197.92 95.38) (width 0.25) (layer F.Cu) (net 3))
-  (segment (start 197.92 95.38) (end 197.92 97.4) (width 0.25) (layer F.Cu) (net 3))
-  (segment (start 197.92 97.4) (end 197.92 98.5) (width 0.25) (layer F.Cu) (net 3))
+  (segment (start 199.98575 93.21425) (end 197.92 95.28) (width 0.25) (layer F.Cu) (net 3))
+  (segment (start 199.98575 89.198055) (end 199.98575 93.21425) (width 0.25) (layer F.Cu) (net 3))
+  (segment (start 197.92 95.28) (end 197.92 97.4) (width 0.25) (layer F.Cu) (net 3))
   (segment (start 204.25 80.8) (end 204.725102 80.8) (width 0.25) (layer F.Cu) (net 4))
   (segment (start 204.725102 80.8) (end 207.1 83.174898) (width 0.25) (layer F.Cu) (net 4))
@@
   (segment (start 222.62 99.62) (end 222.74 99.62) (width 0.25) (layer F.Cu) (net 17))
   (segment (start 217.2 88.4) (end 217.2 94.2) (width 0.25) (layer F.Cu) (net 17))
+  (segment (start 196.55 96) (end 196.55 96.9) (width 0.25) (layer F.Cu) (net 18))
+  (segment (start 196.55 96.9) (end 193.715179 99.734821) (width 0.25) (layer F.Cu) (net 18))
+  (segment (start 193.715179 99.734821) (end 193.265179 99.734821) (width 0.25) (layer F.Cu) (net 18))
   (segment (start 193.8 96.88) (end 197.92 101) (width 0.25) (layer B.Cu) (net 18))
   (segment (start 181.38 84.46) (end 193.8 96.88) (width 0.25) (layer B.Cu) (net 18))
