File: BrainDamage.sch (KiCad schematic (older format))
At the start: 41 parts, among them CON1 AVR-ISP-10, IC1 ATMEGA328P-A, J1 TEST_2P, J2 TEST_2P, J3 TEST_2P, J4 TEST_2P, J5 TEST_2P, J6 TEST_2P, J7 FTDI, J8 Bluetooth, P1 CONN_01X03, P10 CONN_01X03, P11 CONN_01X03, P12 CONN_01X03, P13 CONN_01X03, P14 CONN_01X03, P15 CONN_01X03, P16 CONN_01X03, P17 CONN_01X03, P2 CONN_01X03, P3 CONN_01X03, P4 CONN_01X03, P5 CONN_01X03, P6 CONN_01X03, P7 CONN_01X03, P8 CONN_01X08, P9 CONN_01X03, SW1 SW_PUSH, U1 PCA9685-TSSOP, X1 CRYSTAL_SMD

Commit message: Add files via upload
Parts:
- removed R6: 20K, Resistors_SMD:R_0805_HandSoldering, symbol R
- removed R8: 10K, Resistors_SMD:R_0805_HandSoldering, symbol R
- added C1, C2: C, Capacitors_SMD:C_Trimmer_Murata_TZB4-A, symbol C
- added C3, C6: C, Capacitors_SMD:C_0805_HandSoldering, symbol C
- added C4, C5: 1n, Capacitors_SMD:C_0805_HandSoldering, symbol C
- added J10: Conn_01x02, RC-Battery-Connectors:XT-60_male, symbol Conn_01x02
- added J9: USB_OTG, Connectors:USB_Mini-B, symbol USB_OTG
- added U2: CH340G, Housings_SSOP:SOP-16_4.4x10.4mm_Pitch1.27mm, symbol CH340G
- added U3: AP1117-50, TO_SOT_Packages_SMD:SOT-223-3Lead_TabPin2, symbol AP1117-50
- added X2: CRYSTAL_SMD, Crystals:Resonator_SMD_muRata_SFSKA-3pin_7.9x3.8mm_HandSoldering, symbol CRYSTAL_SMD
- renumbered P16 to S0, P14 to S1, P13 to S10, P12 to S11, P11 to S12, P10 to S13, P9 to S14, P7 to S15, P6 to S2, P5 to S3, P4 to S4, P3 to S5, P2 to S6, P1 to S7, P17 to S8, P15 to S9
Connections:
- net labels added: BATT+
- wire segments 173 -> 209
- no-connect marks 2 -> 9
Other:
- moved on the sheet: CON1, J7, J8, R7, R9, X1

Commit message: Add files via upload
Parts:
- added J11, J12: Conn_01x04, Pin_Headers:Pin_Header_Straight_1x04_Pitch2.54mm, symbol Conn_01x04
- J7: value FTDI -> 15A
- P8: footprint Pin_Headers:Pin_Header_Angled_1x08_Pitch2.54mm -> Pin_Headers:Pin_Header_Straight_1x08_Pitch2.54mm
Connections:
- net labels added: PG
- net labels removed: PD7
- wire segments 209 -> 222
- no-connect marks 9 -> 10
Other:
- moved on the sheet: C4, C5, C6, CON1, D1, D2, J10, J7, J8, J9, R1, R2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

Commit message: Add files via upload
Parts:
- C1, C2, C3, C4, C5, C6: symbol C -> device:C
- CON1: symbol AVR-ISP-10 -> atmel:AVR-ISP-10
- D1, D2: symbol LED-RESCUE-uselessPCB -> BrainDamage-rescue:LED-RESCUE-uselessPCB-RESCUE-BrainDamage
- IC1: symbol ATMEGA328P-A -> BrainDamage-rescue:ATMEGA328P-A-RESCUE-BrainDamage
- J1, J2, J3, J4, J5, J6: symbol TEST_2P -> BrainDamage-rescue:TEST_2P-RESCUE-BrainDamage
- J10: symbol Conn_01x02 -> BrainDamage-rescue:Conn_01x02-RESCUE-BrainDamage
- J11, J12, J8: symbol Conn_01x04 -> BrainDamage-rescue:Conn_01x04-RESCUE-BrainDamage
- J7: footprint Pin_Headers:Pin_Header_Angled_1x05_Pitch2.54mm -> Pin_Headers:Pin_Header_Straight_1x05_Pitch2.54mm; symbol Conn_01x05 -> BrainDamage-rescue:Conn_01x05-RESCUE-BrainDamage
- J9: symbol USB_OTG -> BrainDamage-rescue:USB_OTG-RESCUE-BrainDamage
- P8: symbol CONN_01X08 -> BrainDamage-rescue:CONN_01X08-RESCUE-BrainDamage
- R1, R2: symbol R-RESCUE-uselessPCB -> BrainDamage-rescue:R-RESCUE-uselessPCB-RESCUE-BrainDamage
- R3, R4, R5, R7, R9: symbol R -> device:R
- S0, S1, S10, S11, S12, S13, S14, S15, S2, S3, S4, S5, S6, S7, S8, S9: symbol CONN_01X03 -> BrainDamage-rescue:CONN_01X03-RESCUE-BrainDamage
- SW1: symbol SW_PUSH -> BrainDamage-rescue:SW_PUSH-RESCUE-BrainDamage
- U1: symbol PCA9685-TSSOP -> PCA9685-TSSOP:PCA9685-TSSOP
- U2: symbol CH340G -> ch34x:CH340G
- U3: symbol AP1117-50 -> regul:AP1117-50
- X1, X2: symbol CRYSTAL_SMD -> BrainDamage-rescue:CRYSTAL_SMD-RESCUE-BrainDamage
Connections:
- wire segments 222 -> 276

Commit message: Add files via upload
Parts:
- added C7: 1n, Capacitors_SMD:C_0805_HandSoldering, symbol device:C
Connections:
- wire segments 276 -> 278
- no-connect marks 10 -> 9
Other:
- moved on the sheet: C4, C5, CON1, D1, D2, J11, J12, J7, J8, J9, R1, R2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

Commit message: Add files via upload
Parts:
- added R6: 10K, Resistors_SMD:R_0805_HandSoldering, symbol device:R
Connections:
- wire segments 278 -> 279
Changed lines of the file:
@@
 RESET
 Connection ~ 1200 3950
+$Comp
+L device:R R6
+U 1 1 5A9C29D4
+P 10850 4950
+F 0 "R6" V 10930 4950 50  0000 C CNN
+F 1 "10K" V 10850 4950 50  0000 C CNN
+F 2 "Resistors_SMD:R_0805_HandSoldering" V 10780 4950 50  0001 C CNN
+F 3 "" H 10850 4950 50  0001 C CNN
+	1    10850 4950
+	1    0    0    -1
+$EndComp
+Wire Wire Line
+	10850 4800 10600 4800
+Connection ~ 10600 4800
 $EndSCHEMATC
